File: modbus_LCD_client_6.sch (EAGLE design)
At the start: 32 parts, among them IC4 7805T_H, IC5 ATMEGA328P-PU, J1 9-12V DC CP, Q1 8MHz, Q2 BSS138, Q3 BSS138, U3 BMP180, X1 ISP6IDC

Commit message: Add files via upload
Connections:
- net GND: now also U$2.GND
- net VCC: now also U$2.VCC
Other:
- note added: "used only 3V3 from Arduino Uno board"
- moved on the sheet: C15, C7, IC5, Q1, U$1, U$2

Commit message: Add files via upload
Parts:
- Q1: value 8MHz -> 16MHz
Changed lines of the file:
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@@
 <part name="C9" library="rcl" deviceset="C-EU" device="C025_050-024X070" value="100nF"/>
 <part name="C8" library="rcl" deviceset="C-EU" device="C0805" value="100nF"/>
-<part name="Q1" library="special" deviceset="XTAL" device="" value="8MHz"/>
+<part name="Q1" library="special" deviceset="XTAL" device="" value="16MHz"/>
 <part name="U$1" library="diy-modules" deviceset="RELAY-2-SRD" device=""/>
 <part name="GND9" library="supply1" deviceset="GND" device=""/>

Commit message: Add files via upload
Parts:
- added C2: 18p, resistor:C-EU025-024X044
Connections:
- removed net N$32: IC5.PB6(XTAL1/TOSC1/PCINT6), Q1.2
- net GND: now also C2.2
- net N$17: now also C2.1, IC5.PB6(XTAL1/TOSC1/PCINT6), Q1.2
Changed lines of the file:
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@@
 <part name="GND2" library="supply1" deviceset="GND" device=""/>
 <part name="P+10" library="supply1" deviceset="VCC" device=""/>
+<part name="C2" library="resistor" deviceset="C-EU" device="025-024X044" value="18p"/>
+<part name="GND3" library="supply1" deviceset="GND" device=""/>
 </parts>
 <sheets>
@@
 <instance part="GND2" gate="1" x="-2.54" y="58.42" rot="R180"/>
 <instance part="P+10" gate="VCC" x="-2.54" y="38.1" rot="R180"/>
+<instance part="C2" gate="G$1" x="15.24" y="116.84" rot="R270"/>
+<instance part="GND3" gate="1" x="10.16" y="121.92" rot="R180"/>
 </instances>
 <busses>
@@
 <wire x1="-2.54" y1="50.8" x2="-2.54" y2="55.88" width="0.1524" layer="91"/>
 </segment>
+<segment>
+<pinref part="C2" gate="G$1" pin="2"/>
+<pinref part="GND3" gate="1" pin="GND"/>
+<wire x1="10.16" y1="119.38" x2="10.16" y2="116.84" width="0.1524" layer="91"/>
+</segment>
 </net>
 <net name="N$5" class="0">
@@
 <wire x1="25.4" y1="106.68" x2="17.78" y2="106.68" width="0.1524" layer="91"/>
 </segment>
-</net>
-<net name="N$32" class="0">
-<segment>
+<segment>
+<wire x1="25.4" y1="116.84" x2="17.78" y2="116.84" width="0.1524" layer="91"/>
+<pinref part="C2" gate="G$1" pin="1"/>
 <pinref part="IC5" gate="1" pin="PB6(XTAL1/TOSC1/PCINT6)"/>
 <pinref part="Q1" gate="G$1" pin="2"/>
-<wire x1="35.56" y1="111.76" x2="25.4" y2="116.84" width="0.1524" layer="91"/>
-</segment>
-</net>
+<wire x1="35.56" y1="111.76" x2="35.56" y2="116.84" width="0.1524" layer="91"/>
+<wire x1="35.56" y1="116.84" x2="25.4" y2="116.84" width="0.1524" layer="91"/>
+<junction x="25.4" y="116.84"/>
+</segment>
+</net>
